File: minimouse.kicad_pcb (KiCad board)
At the start: 2 copper layers, 90 x 85 mm, 22 parts, among them J1 Conn_ARM_JTAG_SWD_10, J5 Conn_01x02, M1 N20_encoder, M2 N20_encoder, U1 STM32F030C8Tx, U4 HC-SR04

Commit message: tp3
Parts:
- added C10: 2.2uF, Capacitor_SMD:C_0603_1608Metric, F.Cu at (61.5, 59.3)
- added C11: 2.2uF, Capacitor_SMD:C_0603_1608Metric, F.Cu at (156.0, 72.0)
- added C12: 2.2uF, Capacitor_SMD:C_0603_1608Metric, F.Cu at (128.8, 75.8)
- added C13: 2.2uF, Capacitor_SMD:C_0603_1608Metric, F.Cu at (136.0, 76.0)
- added C7: 2.2uF, Capacitor_SMD:C_0603_1608Metric, F.Cu at (158.8, 99.5)
- added C8: 2.2uF, Capacitor_SMD:C_0603_1608Metric, F.Cu at (115.5, 98.0)
- added C9: 2.2uF, Capacitor_SMD:C_0603_1608Metric, F.Cu at (115.6, 77.0)
- added CEN1: 1 nF / 6.3 V, Capacitor_SMD:C_0603_1608Metric, F.Cu at (177.8, 74.5)
- added CRCOFF1: 22nF, Capacitor_SMD:C_0603_1608Metric, F.Cu at (183.7, 77.0)
- added CS1: 2.2uF, Capacitor_SMD:C_0603_1608Metric, F.Cu at (176.7, 84.4)
- added CSPOL1: 22uF, Capacitor_SMD:C_0603_1608Metric, F.Cu at (176.6, 85.9)
- added CSTBY1: 1 nF, Capacitor_SMD:C_0603_1608Metric, F.Cu at (167.4, 85.8)
- added D1: LED, LED_SMD:LED_0603_1608Metric, F.Cu at (138.3, 79.5)
- added J4: Conn_01x06, Connector_PinHeader_2.54mm:PinHeader_1x06_P2.54mm_Vertical, F.Cu at (164.8, 100.0)
- added J6: Conn_01x04, Connector_PinHeader_2.54mm:PinHeader_1x04_P2.54mm_Vertical, F.Cu at (119.6, 80.4)
- added J7: Conn_01x06, Connector_PinHeader_2.54mm:PinHeader_1x06_P2.54mm_Vertical, F.Cu at (122.2, 100.3)
- added R10: 100, Resistor_SMD:R_0603_1608Metric, F.Cu at (172.3, 96.7)
- added R11: 100, Resistor_SMD:R_0603_1608Metric, F.Cu at (129.8, 96.8)
- added R12: 100, Resistor_SMD:R_0603_1608Metric, F.Cu at (169.9, 96.7)
- added R13: 100, Resistor_SMD:R_0603_1608Metric, F.Cu at (127.3, 96.8)
- added R14: R, Resistor_SMD:R_0603_1608Metric, F.Cu at (138.3, 76.0)
- added R15: 2.2K, Resistor_SMD:R_0603_1608Metric, F.Cu at (183.6, 80.8)
- added R16: 2.2K, Resistor_SMD:R_0603_1608Metric, F.Cu at (183.6, 84.1)
- added R17: 100, Resistor_SMD:R_0603_1608Metric, F.Cu at (160.8, 72.0)
- added REN1: 18K, Resistor_SMD:R_0603_1608Metric, F.Cu at (175.3, 72.2)
- added ROFF1: 47K, Resistor_SMD:R_0603_1608Metric, F.Cu at (180.1, 78.5)
- added RRCOFF1: 1 K, Resistor_SMD:R_0603_1608Metric, F.Cu at (180.1, 77.0)
- added RSNSA1: 33m, Resistor_SMD:R_0603_1608Metric, F.Cu at (172.8, 82.2)
- added RSNSB1: 33m, Resistor_SMD:R_0603_1608Metric, F.Cu at (180.5, 81.8)
- added RSTBY1: 18K, Resistor_SMD:R_0603_1608Metric, F.Cu at (167.4, 82.6)
- added U2: STSPIN240, Package_DFN_QFN:VQFN-16-1EP_3x3mm_P0.5mm_EP1.8x1.8mm, F.Cu at (175.7, 80.5)
- added U3: LP5907MFX-1.2, Package_TO_SOT_SMD:SOT-23-5, F.Cu at (132.4, 76.1)
- moved J1 34.2 mm to (129.9, 86.7)
- moved C4 17.3 mm to (139.2, 91.7)
- moved C5 15.2 mm to (139.1, 93.2)
- moved C2 8.33 mm to (139.2, 88.6), turned to 180 degrees
- moved C6 5.15 mm to (139.0, 85.2), turned to 180 degrees
- moved C3 4.77 mm to (139.2, 90.2)
- moved C1 4.20 mm to (139.1, 86.9)
- moved R5 3.54 mm to (148.5, 96.9)
- moved R4 3.51 mm to (146.9, 96.8)
- moved R3 3.51 mm to (145.4, 96.9)
- moved R2 2.82 mm to (142.4, 92.6), turned to 0 degrees
- moved R7 2.71 mm to (151.5, 96.8)
- moved R6 2.69 mm to (150.0, 96.8)
- moved R1 1.74 mm to (148.5, 79.6), turned to 180 degrees
- moved R9 1.44 mm to (148.0, 82.2)
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Connections:
- U4 pad 4: +3V3 -> +BATT

Commit message: nadjibmarouen
Parts:
- moved C10 105.3 mm to (165.9, 73.0)
- moved C5 19.3 mm to (156.9, 85.5), turned to 90 degrees
- moved REN1 17.7 mm to (179.3, 89.5), turned to 0 degrees
- moved CEN1 17.3 mm to (181.1, 91.6), turned to 0 degrees
- moved CRCOFF1 17.3 mm to (171.0, 88.7), turned to 180 degrees
- moved R3 17.1 mm to (162.3, 94.4), turned to 0 degrees
- moved C9 16.1 mm to (121.4, 91.9)
- moved R4 15.9 mm to (162.3, 92.9), turned to 0 degrees
- moved C1 15.0 mm to (131.2, 74.3)
- moved R5 14.9 mm to (162.3, 91.3), turned to 0 degrees
- moved R6 14.2 mm to (162.3, 89.8), turned to 180 degrees
- moved R7 13.7 mm to (162.3, 88.3), turned to 180 degrees
- moved R8 13.6 mm to (138.8, 88.9), turned to 0 degrees
- moved ROFF1 13.5 mm to (175.1, 91.0), turned to 180 degrees
- moved RRCOFF1 12.8 mm to (174.8, 88.7), turned to 180 degrees
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Connections:
- C12 pad 1: +BATT -> GND
- C12 pad 2: GND -> +BATT
- CS1 pad 1: +3.3V -> +BATT
- CSPOL1 pad 1: +3.3V -> +BATT
- U2 pad 6: +3.3V -> +BATT
- U4 pad 4: +BATT -> +3.3V
Routing:
- net +BATT: track 0.00 -> 119.4 mm
- net +3.3V: track 0.00 -> 72.2 mm
- net Net-(D1-A): track 0.00 -> 2.65 mm
- net GND: track 0.00 -> 2.61 mm
