File: mm_mcu.kicad_sch (KiCad schematic)
At the start: 18 parts, among them J1 Conn_ARM_JTAG_SWD_10, U1 STM32F030C8Tx

Commit message: tp2_connection
Parts:
- added M1 (x2): N20_encoder, minimouse:N20_with_encoder, symbol minimouse:N20_w_encoder
Changed lines of the file:
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@@
+    (stroke (width 0) (type default))
+  )
+  (wire (pts (xy 77.47 83.82) (xy 77.47 86.36))
+    (stroke (width 0) (type default))
+  )
+  (wire (pts (xy 77.47 86.36) (xy 74.93 86.36))
     (stroke (width 0) (type default))
   )
@@
     (stroke (width 0) (type default))
   )
+  (wire (pts (xy 81.28 102.87) (xy 82.55 102.87))
+    (stroke (width 0) (type default))
+  )
   (wire (pts (xy 220.98 27.94) (xy 229.87 27.94))
     (stroke (width 0) (type default))
@@
     (stroke (width 0) (type default))
   )
+  (wire (pts (xy 82.55 100.33) (xy 81.28 100.33))
+    (stroke (width 0) (type default))
+  )
   (wire (pts (xy 81.28 46.99) (xy 88.9 46.99))
     (stroke (width 0) (type default))
@@
     (stroke (width 0) (type default))
   )
+  (wire (pts (xy 115.57 111.76) (xy 115.57 105.41))
+    (stroke (width 0) (type default))
+  )
   (wire (pts (xy 256.54 39.37) (xy 247.65 39.37))
     (stroke (width 0) (type default))
@@
     (stroke (width 0) (type default))
   )
+  (wire (pts (xy 77.47 83.82) (xy 74.93 83.82))
+    (stroke (width 0) (type default))
+  )
   (wire (pts (xy 139.7 120.65) (xy 139.7 123.19))
     (stroke (width 0) (type default))
@@
     (stroke (width 0) (type default))
   )
+  (wire (pts (xy 82.55 102.87) (xy 82.55 100.33))
+    (stroke (width 0) (type default))
+  )
+  (wire (pts (xy 113.03 111.76) (xy 115.57 111.76))
+    (stroke (width 0) (type default))
+  )
   (wire (pts (xy 62.23 156.21) (xy 69.85 156.21))
     (stroke (width 0) (type default))
@@
   )
   (hierarchical_label "UART1_RX" (shape input) (at 97.79 92.71 180) (fields_autoplaced)
+    (effects (font (size 1.27 1.27)) (justify right))
+  )
+  (hierarchical_label "C1" (shape output) (at 81.28 100.33 180) (fields_autoplaced)
     (effects (font (size 1.27 1.27)) (justify right))
   )
@@
     (effects (font (size 1.27 1.27)) (justify right))
   )
+  (hierarchical_label "C2" (shape output) (at 78.74 92.71 180) (fields_autoplaced)
+    (effects (font (size 1.27 1.27)) (justify right))
+  )
   (hierarchical_label "IN_B2" (shape output) (at 97.79 80.01 180) (fields_autoplaced)
     (effects (font (size 1.27 1.27)) (justify right))
@@
     (effects (font (size 1.27 1.27)) (justify left))
   )
+  (hierarchical_label "C2" (shape output) (at 78.74 92.71 180) (fields_autoplaced)
+    (effects (font (size 1.27 1.27)) (justify right))
+  )
   (hierarchical_label "OUT_A4" (shape output) (at 182.88 52.07 0) (fields_autoplaced)
     (effects (font (size 1.27 1.27)) (justify left))
   )
+  (hierarchical_label "C1" (shape output) (at 81.28 102.87 180) (fields_autoplaced)
+    (effects (font (size 1.27 1.27)) (justify right))
+  )
   (hierarchical_label "OUT_B1" (shape output) (at 97.79 77.47 180) (fields_autoplaced)
+    (effects (font (size 1.27 1.27)) (justify right))
+  )
+  (hierarchical_label "MB" (shape passive) (at 115.57 105.41 180) (fields_autoplaced)
+    (effects (font (size 1.27 1.27)) (justify right))
+  )
+  (hierarchical_label "MA" (shape passive) (at 74.93 86.36 180) (fields_autoplaced)
     (effects (font (size 1.27 1.27)) (justify right))
   )
@@
     (effects (font (size 1.27 1.27)) (justify right))
   )
+  (hierarchical_label "MA" (shape passive) (at 74.93 83.82 180) (fields_autoplaced)
+    (effects (font (size 1.27 1.27)) (justify right))
+  )
   (hierarchical_label "TIM15_CH2" (shape output) (at 182.88 49.53 0) (fields_autoplaced)
     (effects (font (size 1.27 1.27)) (justify left))
+  )
+  (hierarchical_label "MB" (shape passive) (at 113.03 111.76 180) (fields_autoplaced)
+    (effects (font (size 1.27 1.27)) (justify right))
   )
   (hierarchical_label "TIM3_CH2" (shape input) (at 182.88 59.69 0) (fields_autoplaced)
@@
   )
   (symbol (lib_id "Connector:Conn_ARM_JTAG_SWD_10") (at 49.53 163.83 0) (unit 1)
-    (in_bom yes) (on_board yes) (dnp no) (fields_autoplaced)
+    (in_bom yes) (on_board yes) (dnp no)
     (property "Reference" "J1" (at 38.1 162.56 0)
       (effects (font (size 1.27 1.27)) (justify right))
     )
-    (property "Value" "Conn_ARM_JTAG_SWD_10" (at 38.1 165.1 0)
+    (property "Value" "Conn_ARM_JTAG_SWD_10" (at 36.83 166.37 0)
       (effects (font (size 1.27 1.27)) (justify right))
     )
@@
         (path "/d8fa4cba-2469-4231-847f-065b6b829f44/b5d7e952-00af-4b6f-924a-ee43c62726d2"
           (reference "J1") (unit 1)
+        )
+      )
+    )
+  )
+  (symbol (lib_id "minimouse:N20_w_encoder") (at 104.14 58.42 0) (unit 1)
+    (in_bom yes) (on_board yes) (dnp no) (fields_autoplaced)
+    (property "Reference" "M1" (at 106.68 57.15 0)
+      (effects (font (size 1.27 1.27)) (justify left))
+    )
+    (property "Value" "N20_encoder" (at 106.68 59.69 0)
+      (effects (font (size 1.27 1.27)) (justify left))
+    )
+    (property "Footprint" "minimouse:N20_with_encoder" (at 106.68 54.61 0)
+      (effects (font (size 1.27 1.27)) hide)
+    )
+    (property "Datasheet" "" (at 104.14 58.42 0)
+      (effects (font (size 1.27 1.27)) hide)
+    )
+    (instances
+      (project "minimouse"
+        (path "/d8fa4cba-2469-4231-847f-065b6b829f44/7f113667-692a-4f4d-b16f-621d32f3f136"
+          (reference "M1") (unit 1)
+        )
+        (path "/d8fa4cba-2469-4231-847f-065b6b829f44/3975acd0-18ad-47bc-9ce1-d8c4d864aafe"
+          (reference "M2") (unit 1)
+        )
+        (path "/d8fa4cba-2469-4231-847f-065b6b829f44/b5d7e952-00af-4b6f-924a-ee43c62726d2"
+          (reference "M1") (unit 1)
         )
       )
@@
         )
       )
+    )
+  )
+  (symbol (lib_id "minimouse:N20_w_encoder") (at 104.14 58.42 0) (unit 1)
+    (in_bom yes) (on_board yes) (dnp no) (fields_autoplaced)
+    (property "Reference" "M1" (at 106.68 57.15 0)
+      (effects (font (size 1.27 1.27)) (justify left))
+    )
+    (property "Value" "N20_encoder" (at 106.68 59.69 0)
+      (effects (font (size 1.27 1.27)) (justify left))
+    )
+    (property "Footprint" "minimouse:N20_with_encoder" (at 106.68 54.61 0)
+      (effects (font (size 1.27 1.27)) hide)
+    )
+    (property "Datasheet" "" (at 104.14 58.42 0)
+      (effects (font (size 1.27 1.27)) hide)
+    )
+    (instances
+      (project "minimouse"
+        (path "/d8fa4cba-2469-4231-847f-065b6b829f44/7f113667-692a-4f4d-b16f-621d32f3f136"
+          (reference "M1") (unit 1)
+        )
+        (path "/d8fa4cba-2469-4231-847f-065b6b829f44/3975acd0-18ad-47bc-9ce1-d8c4d864aafe"
+          (reference "M2") (unit 1)
+        )
+        (path "/d8fa4cba-2469-4231-847f-065b6b829f44/b5d7e952-00af-4b6f-924a-ee43c62726d2"
+          (reference "M1") (unit 1)
+        )
+      )

Commit message: nadjibmarouen
Parts:
- removed M1 (x2): N20_encoder, minimouse:N20_with_encoder, symbol minimouse:N20_w_encoder
Changed lines of the file:
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@@
-    )
-  )
-  (symbol (lib_id "minimouse:N20_w_encoder") (at 104.14 58.42 0) (unit 1)
-    (in_bom yes) (on_board yes) (dnp no) (fields_autoplaced)
-    (property "Reference" "M1" (at 106.68 57.15 0)
-      (effects (font (size 1.27 1.27)) (justify left))
-    )
-    (property "Value" "N20_encoder" (at 106.68 59.69 0)
-      (effects (font (size 1.27 1.27)) (justify left))
-    )
-    (property "Footprint" "minimouse:N20_with_encoder" (at 106.68 54.61 0)
-      (effects (font (size 1.27 1.27)) hide)
-    )
-    (property "Datasheet" "" (at 104.14 58.42 0)
-      (effects (font (size 1.27 1.27)) hide)
-    )
-    (instances
-      (project "minimouse"
-        (path "/d8fa4cba-2469-4231-847f-065b6b829f44/7f113667-692a-4f4d-b16f-621d32f3f136"
-          (reference "M1") (unit 1)
-        )
-        (path "/d8fa4cba-2469-4231-847f-065b6b829f44/3975acd0-18ad-47bc-9ce1-d8c4d864aafe"
-          (reference "M2") (unit 1)
-        )
-        (path "/d8fa4cba-2469-4231-847f-065b6b829f44/b5d7e952-00af-4b6f-924a-ee43c62726d2"
-          (reference "M1") (unit 1)
-        )
-      )
     )
   )
@@
         )
       )
-    )
-  )
-  (symbol (lib_id "minimouse:N20_w_encoder") (at 104.14 58.42 0) (unit 1)
-    (in_bom yes) (on_board yes) (dnp no) (fields_autoplaced)
-    (property "Reference" "M1" (at 106.68 57.15 0)
-      (effects (font (size 1.27 1.27)) (justify left))
-    )
-    (property "Value" "N20_encoder" (at 106.68 59.69 0)
-      (effects (font (size 1.27 1.27)) (justify left))
-    )
-    (property "Footprint" "minimouse:N20_with_encoder" (at 106.68 54.61 0)
-      (effects (font (size 1.27 1.27)) hide)
-    )
-    (property "Datasheet" "" (at 104.14 58.42 0)
-      (effects (font (size 1.27 1.27)) hide)
-    )
-    (instances
-      (project "minimouse"
-        (path "/d8fa4cba-2469-4231-847f-065b6b829f44/7f113667-692a-4f4d-b16f-621d32f3f136"
-          (reference "M1") (unit 1)
-        )
-        (path "/d8fa4cba-2469-4231-847f-065b6b829f44/3975acd0-18ad-47bc-9ce1-d8c4d864aafe"
-          (reference "M2") (unit 1)
-        )
-        (path "/d8fa4cba-2469-4231-847f-065b6b829f44/b5d7e952-00af-4b6f-924a-ee43c62726d2"
-          (reference "M1") (unit 1)
-        )
-      )
