File: mm_motor_control.kicad_sch (KiCad schematic)
At the start: 0 parts

Commit message: tp2_connection
Parts:
- added CEN: 1 nF / 6.3 V, symbol Device:C
- added CRCOFF: 22nF, symbol Device:C
- added CS: 2.2uF, symbol Device:C
- added CSPOL: 22uF, symbol Device:C
- added CSTBY: 1 nF, symbol Device:C
- added R (x2): 2.2K, symbol Device:R
- added REN, RSTBY: 18K, symbol Device:R
- added ROFF: 47K, symbol Device:R
- added RRCOFF: 1 K, symbol Device:R
- added RSNSA, RSNSB: 33m, symbol Device:R
- added U2: STSPIN240, Package_DFN_QFN:VQFN-16-1EP_3x3mm_P0.5mm_EP1.8x1.8mm, symbol Driver_Motor:STSPIN240
Connections:
- net EN: now also CEN.1, REN.2, U2.13 (EN/FLT)
- net FAULT: now also REN.1
- net OUT_A1: now also U2.3 (OUTA1)
- net OUT_A2: now also U2.5 (OUTA2)
- net OUT_B1: now also U2.10 (OUTB1)
- net OUT_B2: now also U2.8 (OUTB2)
- net PHASE_A: now also U2.1 (PHA)
- net PHASE_B: now also U2.15 (PHB)
- net PWM_A: now also U2.2 (PWMA)
- net PWM_B: now also U2.16 (PWMB)
- net STBY/RESET: now also CSTBY.1, RSTBY.2, U2.14 (STBY/RESET)
- new net: RSNSB.1, U2.9 (SENSEB)
- new net: R.1, R.2, U2.11 (REF)
- new net: CRCOFF.1, RRCOFF.2
- new net: ROFF.1, RRCOFF.1, U2.12 (TOFF)
- new net: RSNSA.1, U2.4 (SENSEA)
- new net +3.3V: CS.1, CSPOL.1, RSTBY.1, U2.6 (VS)
- new net +BATT: R.1
- new net GND: CEN.2, CRCOFF.2, CS.2, CSPOL.2, CSTBY.2, R.2, ROFF.2, RSNSA.2, RSNSB.2, U2.17 (EPAD), U2.7 (GND)

Commit message: nadjibmarouen
Parts:
- added C8: 2.2uF, Capacitor_SMD:C_0603_1608Metric, symbol Device:C
- CEN1: renamed from CEN; footprint (none) -> Capacitor_SMD:C_0603_1608Metric
- CRCOFF1: renamed from CRCOFF; footprint (none) -> Capacitor_SMD:C_0603_1608Metric
- CS1: renamed from CS; footprint (none) -> Capacitor_SMD:C_0603_1608Metric
- CSPOL1: renamed from CSPOL; footprint (none) -> Capacitor_SMD:C_0603_1608Metric
- CSTBY1: renamed from CSTBY; footprint (none) -> Capacitor_SMD:C_0603_1608Metric
- R15, R16: renamed from R; footprint (none) -> Resistor_SMD:R_0603_1608Metric
- REN1: renamed from REN; footprint (none) -> Resistor_SMD:R_0603_1608Metric
- ROFF1: renamed from ROFF; footprint (none) -> Resistor_SMD:R_0603_1608Metric
- RRCOFF1: renamed from RRCOFF; footprint (none) -> Resistor_SMD:R_0603_1608Metric
- RSNSA1: renamed from RSNSA; footprint (none) -> Resistor_SMD:R_0603_1608Metric
- RSNSB1: renamed from RSNSB; footprint (none) -> Resistor_SMD:R_0603_1608Metric
- RSTBY1: renamed from RSTBY; footprint (none) -> Resistor_SMD:R_0603_1608Metric
Connections:
- net +BATT: now also C8.1
- net GND: now also C8.2
